Commit message: Remove ft legs from model ergocub

File: urdf/ergoCub/robots/ergoCubSN000/model.urdf (robot description, URDF)
Before this commit: robot ergoCub, 194 links, 193 joints
Joints:
- removed joint l_leg_ft_sensor
- removed joint r_leg_ft_sensor
- added joint l_leg_ft_joint: type fixed, parent l_hip_2, child l_hip_3, origin xyz=0.036699999999999997 0 -0.0897 rpy=0 0 0
- added joint r_leg_ft_joint: type fixed, parent r_hip_2, child r_hip_3, origin xyz=0.036699999999999997 0 -0.0897 rpy=0 0 0
- joint torso_pitch: origin xyz=0 0 0.11800000000000005 rpy=0 0.174533 0 -> xyz=0 0 0.11800000000000005 rpy=0 0 0; type fixed -> revolute
